Commit message: refactor: update robot model initialization with mesh directories, and adjust test plotting.

File: classes/robots/robot_models/softleg_urdf/urdf/leg_constrained.urdf (robot description, URDF)
Before this commit: robot leg_constrained, 6 links, 5 joints
Links:
- link LH_LOWER_LEG: geometry collision box size=0.269 0.057 0.060; visual mesh filename=Lower_leg_left.stl
- link LH_SHOULDER: geometry collision box size=0.269 0.057 0.060; visual mesh filename=Module_left_hind.stl
- link LH_UPPER_LEG: geometry collision box size=0.269 0.057 0.060; visual mesh filename=Module_left_hind.stl
- link base_link: geometry visual mesh filename=cart.stl scale=0.001 0.001 0.001
